File: hardware/mini-sumo.kicad_sch (KiCad schematic)
At the start: 76 parts, among them J1 IR Sensor 1, J11 BATTERY, J12 MOTOR1, J13 MOTOR2, J14 Conn_02x03_Counter_Clockwise, J2 IR Sensor 2, J3 IR Sensor 5, J4 IR Sensor 4, J5 IR LED, J6 Floor Sensor 1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

Commit message: Finalized the PCB
Parts:
- removed J14: Conn_02x03_Counter_Clockwise, Connector_PinHeader_2.54mm:PinHeader_2x03_P2.54mm_Vertical, symbol Connector_Generic:Conn_02x03_Counter_Clockwise
- added J10: Conn_02x03_Odd_Even, Connector_PinHeader_2.54mm:PinHeader_2x03_P2.54mm_Vertical, symbol Connector_Generic:Conn_02x03_Odd_Even
- VD1: footprint Diodes_THT:D_DO-35_SOD27_P2.54mm_Vertical_AnodeUp -> Diode_THT:D_DO-35_SOD27_P2.54mm_Vertical_AnodeUp
- renumbered SW2 to SW1, SW3 to SW2, SW4 to SW3, SW5 to SW4
Connections:
- net +3V3: now also J10.2 (Pin_2)
- net GND: now also J10.6 (Pin_6)
- net GPIO38: now also J10.5 (Pin_5)
- net GPIO39: now also J10.3 (Pin_3)
- net GPIO40: now also J10.1 (Pin_1)
- net GPIO41: now also J10.4 (Pin_4)

Commit message: Improved sikscreen on PCB. Changed reverse polarity transistor to AO3401A.
Parts:
- VT3: value FDN360P -> AO3401A
Changed lines of the file:
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@@
 			)
 		)
-		(property "Value" "FDN360P"
+		(property "Value" "AO3401A"
 			(at 266.7 145.415 0)
 			(effects

Commit message: Organized and fixed schematic. Added schematic PDF and HTML interactive BOM.
Parts:
- BZ1: LCSC Part (none) -> C2693577
- C1, C2, C3, C4: LCSC Part (none) -> C5632433
- C10, C12, C14, C15, C6, C7, C8: LCSC Part (none) -> C5632430
- C11, C13: value 10uF -> 100uF; LCSC Part (none) -> C44588
- C16: value 10uF -> 47uF; LCSC Part (none) -> C13654
- C5, C9: value 0.1uF -> 1uF; LCSC Part (none) -> C5632434
- D1: value 1N5819 -> 1N5817; LCSC Part (none) -> C7544876
- DA1: LCSC Part (none) -> C347222
- DA2: LCSC Part (none) -> C347224
- J1, J2, J4, J6, J8: LCSC Part (none) -> C722936
- J10: now not fitted
- J11, J12, J13: LCSC Part (none) -> C7429542
- J3: value IR Sensor 5 -> IR Sensor 3; LCSC Part (none) -> C722936
- J5, J7: LCSC Part (none) -> C722910
- J9: LCSC Part (none) -> C722918
- R1, R10, R12, R7: LCSC Part (none) -> C119858
- R11, R21, R23, R6: LCSC Part (none) -> C119870
- R13, R15, R16, R19, R22, R8: LCSC Part (none) -> C714232
- R14, R9: LCSC Part (none) -> C119195
- R17, R18: value 33R -> 22R; LCSC Part (none) -> C119830
- R2, R3, R4, R5: LCSC Part (none) -> C2896920
- R20: value 10k -> 4k7; LCSC Part (none) -> C714232
- R24: LCSC Part (none) -> C119862
- SW2, SW3, SW4: LCSC Part (none) -> C2845253
- U10, U3, U5, U6, U7, U9: LCSC Part (none) -> C2843785
- VD1: LCSC Part (none) -> C5158978
- VT1, VT2, VT4: LCSC Part (none) -> C713610
- VT3: LCSC Part (none) -> C15127
Other:
- note added: "Accelerometer"
- note added: "Buttons"
- note added: "Extra GPIOs"
- note added: "Floor sensors"
- note added: "IR LED drivers"
- note added: "LED Power"
- note added: "Microcontroller"
- note added: "Motor driver"
- note added: "Opponent sensors"
- note added: "Power"
- note added: "RGB LEDs"
- note added: "Reset"
- note added: "ToF sensor connector"
- note added: "USB-C"
- note removed: "3-4x Floor sensor 3-4x ADC (3-4 pins) 3x Laser sensor - I2C SDA & SCL + 3x out + 3x in (8 pins) 1x IR remote RX (1 pin) 1x IR remote TX? (1 pin) 5x IR sensors + 1x TX pin (6 pins) 2x motor control 2 pins per motor (4 pins) 1x gyro - I2C + Int (3 pins) 1x buzzer (1 pin) 1x WS2812B (1 pin) 2x buttons (2 pins) 1x oled I2C (2 pins) Total: 33"
- note removed: "3x Floor sensor 3x ADC (3 pins) 1x Laser sensor - I2C SDA & SCL + 1x out + 1x in (4 pins) 1x IR remote RX (1 pin) 3x IR sensors + 1x TX pin (4 pins) 2x motor control 2 pins per motor (4 pins) 1x gyro - I2C + Int (3 pins) 1x buzzer (1 pin) 1x WS2812B (1 pin) 2x buttons (2 pins) Total: 23"
- company: (none) -> RV1G Robotics Club
- title: (none) -> Mini Sumo
- moved on the sheet: BZ1, C1, C10, C11, C12, C13, C14, C15, C16, C2, C3, C4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
